Commit message: new aliengo urdf without third camera looking to the floor

File: aliengolib/aliengo.urdf (robot description, URDF)
Before this commit: robot aliengo, 51 links, 50 joints
Links:
- removed link realsense/down/camera_bottom_screw_frame
- removed link realsense/down/camera_color_frame
- removed link realsense/down/camera_color_optical_frame
- removed link realsense/down/camera_depth_frame
- removed link realsense/down/camera_depth_optical_frame
- removed link realsense/down/camera_left_ir_frame
- removed link realsense/down/camera_left_ir_optical_frame
- removed link realsense/down/camera_link
- removed link realsense/down/camera_right_ir_frame
- removed link realsense/down/camera_right_ir_optical_frame
Joints:
- removed joint realsense/down/camera_color_joint
- removed joint realsense/down/camera_color_optical_joint
- removed joint realsense/down/camera_depth_joint
- removed joint realsense/down/camera_depth_optical_joint
- removed joint realsense/down/camera_left_ir_joint
- removed joint realsense/down/camera_left_ir_optical_joint
- removed joint realsense/down/camera_link_joint
- removed joint realsense/down/camera_right_ir_joint
- removed joint realsense/down/camera_right_ir_optical_joint
- removed joint realsense/down/trunkcamera_joint
